Commit message: robot staet publiher

File: src/my_robot/description/my_robot_core.xacro (robot description, xacro)
@@ -4,4 +4,5 @@
     <xacro:property name="chassis_width" value="0.3"/>
     <xacro:property name="chassis_height" value="0.15"/>
+    <xacro:include filename="inertial_macros.xacro"/>
     <material name="white">
         <color rgba="1 1 1 1"/>
@@ -19,4 +20,5 @@
         <color rgba="0 0 1 1"/>
     </material>
+    <!--base link-->
     <link name="base_link">
     </link>
@@ -26,4 +28,5 @@
         <origin xyz="-0.1 0 0"/>
     </joint>
+    <!--chassis link-->
     <link name="chassis_link">
         <visual>
@@ -40,9 +43,75 @@
             </geometry>
         </collision>
-        <inertial>
+        <xacro:inertial_box mass="0.5" x="${chassis_length}" y="${chassis_width}" z="${chassis_height}">
             <origin xyz="0.15 0 0.075" rpy="0 0 0"/>
-            <mass value="0.5"/>
-            <inertia ixx="0.0046875" ixy="0.0" ixz="0.0" iyy="0.0046875" iyz="0.0" izz="0.0075"/>
-        </inertial>
+        </xacro:inertial_box>
     </link>
+    <!--LEFTWHEEL LINK-->
+    <link name="left_wheel_link">
+        <visual>
+            <geometry>
+                <cylinder radius="0.05" length="0.05"/>
+            </geometry>
+            <material name="black"/>
+        </visual>
+        <collision>
+            <geometry>
+                <cylinder radius="0.05" length="0.05"/>
+            </geometry>
+        </collision>
+        <xacro:inertial_cylinder mass="0.01" length="0.05" radius="0.05">
+            <origin xyz="0 0 0" rpy="0 0 0"/>
+        </xacro:inertial_cylinder>
+    </link>
+    <joint name="left_wheel_joint" type="continuous">
+        <parent link="base_link"/>
+        <child link="left_wheel_link"/>
+        <origin xyz="0 0.175 0" rpy="-1.5708 0 0"/>
+        <axis xyz="0 0 1"/>
+    </joint>
+    <!--right wheel link-->
+    <link name="right_wheel_link">
+        <visual>
+            <geometry>
+                <cylinder radius="0.05" length="0.05"/>
+            </geometry>
+            <material name="black"/>
+        </visual>
+        <collision>
+            <geometry>
+                <cylinder radius="0.05" length="0.05"/>
+            </geometry>
+        </collision>
+        <xacro:inertial_cylinder mass="0.01" length="0.05" radius="0.05">
+            <origin xyz="0 0 0" rpy="0 0 0"/>
+        </xacro:inertial_cylinder>
+    </link>
+    <joint name="right_wheel_joint" type="continuous">
+        <parent link="base_link"/>
+        <child link="right_wheel_link"/>
+        <origin xyz="0 -0.175 0" rpy="1.5708 0 0"/>
+        <axis xyz="0 0 1"/>
+    </joint>
+    <!-- chaster wheel joint -->
+    <link name="caster_wheel_link">
+        <visual>
+            <geometry>
+                <sphere radius="0.05"/>
+            </geometry>
+            <material name="black"/>
+        </visual>
+        <collision>
+            <geometry>
+                <sphere radius="0.05"/>
+            </geometry>
+        </collision>
+        <xacro:inertial_sphere mass="0.01" radius="0.05">
+            <origin xyz="0 0 0" rpy="0 0 0"/>
+        </xacro:inertial_sphere>
+    </link>
+    <joint name="caster_wheel_joint" type="fixed">
+        <parent link="chassis_link"/>
+        <child link="caster_wheel_link"/>
+        <origin xyz="0.25 0 0" rpy="0 0 0"/>
+    </joint>
 </robot>
