Commit message: camera added but not plugin and lidar scan is from origin

File: src/my_robot/description/lidar.xacro (robot description, xacro)
@@ -4,5 +4,5 @@
         <parent link="base_link"/>
         <child link="lidar_link"/>
-        <origin xyz="0.22 0 0.175" rpy="0 0 0"/>
+        <origin xyz="0.14 0 0.175" rpy="0 0 0"/>
     </joint>
     <link name="lidar_link">
@@ -55,9 +55,3 @@
         </sensor>
     </gazebo>
-    <gazebo>
-        <plugin filename="gz-sim-sensors-system" name="gz::sim::systems::Sensors">
-        <render_engine>ogre2</render_engine>
-        <rendering_system>ogre2</rendering_system>
-        </plugin>
-    </gazebo>
 </robot>

File: src/my_robot/description/my_robot.urdf.xacro (robot description, xacro)
@@ -4,3 +4,4 @@
     <xacro:include filename="gz_control.xacro"/>
     <xacro:include filename="lidar.xacro"/>
+    <xacro:include filename="camera.xacro"/>
 </robot>
