Commit message: camera fixed and lidar thing is fixed biut issue is with the gazbo visualizing but in rviz everything is good

File: src/my_robot/description/camera.xacro (robot description, xacro)
@@ -30,25 +30,8 @@
         <origin xyz="0 0 0" rpy="${-pi/2} 0 ${pi/2}"/>
     </joint>
-    <gazebo reference="camera_link_optical">
-        <material>Gazebo/Red</material>
+    <gazebo reference="camera_link">
         <sensor name="camera" type="camera">
-            <pose relative_to="camera_link_optical"> 0 0 0 0 0 0 </pose>
-            <topic>camera/image_raw</topic>
-            <visualize>true</visualize>
-            <always_on>true</always_on>
-            <update_rate>10</update_rate>
             <camera>
-                <horizontal>
-                    <samples>640</samples>
-                    <resolution>1</resolution>
-                    <min_angle>-1.5708</min_angle>
-                    <max_angle>1.5708</max_angle>
-                </horizontal>
-                <vertical>
-                    <samples>480</samples>
-                    <resolution>1</resolution>
-                    <min_angle>-0.7854</min_angle>
-                    <max_angle>0.7854</max_angle>
-                </vertical>
+                <horizontal_fov>1.3962634</horizontal_fov>
                 <image>
                     <width>640</width>
@@ -57,11 +40,22 @@
                 </image>
                 <clip>
-                    <near>0.05</near>
-                    <far>8.0</far>
+                    <near>0.1</near>
+                    <far>15</far>
                 </clip>
+                <noise>
+                    <type>gaussian</type>
+                    <!-- Noise is sampled independently per pixel on each frame.
+                    That pixel's noise value is added to each of its color
+                    channels, which at that point lie in the range [0,1]. -->
+                    <mean>0.0</mean>
+                    <stddev>0.007</stddev>
+                </noise>
+                <optical_frame_id>camera_link_optical</optical_frame_id>
+                <camera_info_topic>camera/camera_info</camera_info_topic>
             </camera>
-            <plugin name="camera_controller" filename="libgazebo_ros_camera.so">
-                <frame_name>camera_link_optical</frame_name>
-            </plugin>
+            <always_on>1</always_on>
+            <update_rate>20</update_rate>
+            <visualize>true</visualize>
+            <topic>camera/image</topic>
         </sensor>
     </gazebo>

File: src/my_robot/description/lidar.xacro (robot description, xacro)
@@ -1,45 +1,60 @@
 <?xml version="1.0"?>
 <robot xmlns:xacro="http://www.ros.org/wiki/xacro">
-    <joint name="lidar_joint" type="fixed">
-        <parent link="base_link"/>
+    <joint type="fixed" name="lidar_joint">
+        <origin xyz="0.15 0 0.185" rpy="0 0 0"/>
         <child link="lidar_link"/>
-        <origin xyz="0.14 0 0.175" rpy="0 0 0"/>
+        <parent link="chassis_link"/>
+        <axis xyz="0 1 0"/>
     </joint>
-    <link name="lidar_link">
-        <visual>
+    <gazebo reference="lidar_joint">
+        <preserveFixedJoint>true</preserveFixedJoint>
+    </gazebo>
+    <link name='lidar_link'>
+        <inertial>
+            <mass value="0.1"/>
+            <origin xyz="0 0 0" rpy="0 0 0"/>
+            <inertia
+                ixx="1e-3" ixy="0" ixz="0"
+                iyy="1e-3" iyz="0"
+                izz="1e-3"
+            />
+        </inertial>
+        <visual name='lidar_link_visual'>
+            <origin xyz="0 0 0" rpy="0 0 0"/>
             <geometry>
-                <cylinder radius="0.05" length="0.05"/>
+                <mesh filename = "package://my_robot/meshes/lidar.dae"/>
             </geometry>
-            <material name="red"/>
         </visual>
         <collision>
+            <origin xyz="0 0 0" rpy="0 0 0"/>
             <geometry>
                 <cylinder radius="0.05" length="0.05"/>
             </geometry>
         </collision>
-        <xacro:inertial_cylinder mass="0.1" radius="0.05" length="0.05">
-            <origin xyz="0 0 0" rpy="0 0 0"/>
-        </xacro:inertial_cylinder>
     </link>
     <gazebo reference="lidar_link">
-        <material>Gazebo/Red</material>
         <sensor name="gpu_lidar" type="gpu_lidar">
+            <pose relative_to="lidar_link"> 0 0 0 0 0 0 </pose>
+            <visualize>true</visualize>
+            <update_rate>10</update_rate>
             <topic>scan</topic>
-            <pose relative_to="lidar_link"> 0 0 0 0 0 0 </pose>
-            <always_on>true</always_on>
-            <visualize>true</visualize>
-            <update_rate>1</update_rate>
             <gz_frame_id>lidar_link</gz_frame_id>
             <lidar>
                 <scan>
                     <horizontal>
-                    <samples>720</samples>
-                    <resolution>1</resolution>
-                    <min_angle>-3.14</min_angle>
-                    <max_angle>3.14</max_angle>
+                        <samples>640</samples>
+                        <resolution>1</resolution>
+                        <min_angle>-3.14159</min_angle>
+                        <max_angle>3.14159</max_angle>
                     </horizontal>
+                    <!-- <vertical>
+                        <samples>16</samples>
+                        <resolution>1</resolution>
+                        <min_angle>-0.261799</min_angle>
+                        <max_angle>0.261799</max_angle>
+                    </vertical> -->
                 </scan>
                 <range>
-                    <min>0.05</min>
+                    <min>0.08</min>
                     <max>10.0</max>
                     <resolution>0.01</resolution>
@@ -47,10 +62,8 @@
                 <noise>
                     <type>gaussian</type>
-                    <mean>0.0</mean>
+                    <mean>0</mean>
                     <stddev>0.01</stddev>
                 </noise>
-                <frame_id>lidar_link</frame_id>
             </lidar>
-            <always_on>1</always_on>
         </sensor>
     </gazebo>

Commit message: added a custom world for auo nav

File: src/my_robot/description/camera.xacro (robot description, xacro)
@@ -52,10 +52,10 @@
                 </noise>
                 <optical_frame_id>camera_link_optical</optical_frame_id>
-                <camera_info_topic>camera/camera_info</camera_info_topic>
+                <camera_info_topic>/camera/camera_info</camera_info_topic>
             </camera>
             <always_on>1</always_on>
             <update_rate>20</update_rate>
             <visualize>true</visualize>
-            <topic>camera/image</topic>
+            <topic>/camera/image</topic>
         </sensor>
     </gazebo>

File: src/my_robot/description/lidar.xacro (robot description, xacro)
@@ -38,5 +38,5 @@
             <visualize>true</visualize>
             <update_rate>10</update_rate>
-            <topic>scan</topic>
+            <topic>/scan</topic>
             <gz_frame_id>lidar_link</gz_frame_id>
             <lidar>

File: src/my_robot/description/my_robot_core.xacro (robot description, xacro)
@@ -23,4 +23,12 @@
     <link name="base_link">
     </link>
+    <!-- base_foot_print -->
+    <link name="base_footprint">
+    </link>
+    <joint name="base_footprint_joint" type="fixed">
+        <parent link="base_link"/>
+        <child link="base_footprint"/>
+        <origin xyz="0 0 0"/>
+    </joint>
     <joint name="chassis_joint" type="fixed">
         <parent link="base_link"/>
